Commit message: Have a map functioning based on lidar odometry

File: autonomous_litter_bot_package/urdf/robot.urdf (robot description, URDF)
Before this commit: robot robot, 4 links, 3 joints
Links:
- removed link lidar
- added link laser; visual cylinder length=0.05 radius=0.04
Joints:
- removed joint body_to_lidar
- removed joint lidar_to_imu
- added joint body_to_laser_frame: type fixed, parent base_link, child laser, origin xyz=0 0.18 -0.075 rpy=3.14159 0 0
- added joint laser_frame_to_imu: type fixed, parent laser, child imu, origin xyz=0 -0.05 0

Commit message: LiDAR and IMU Fused. Correct Orientation with X Forward. EKF filter publishing. Map Generating.

File: autonomous_litter_bot_package/urdf/robot.urdf (robot description, URDF)
Before this commit: robot robot, 4 links, 3 joints
Links:
- removed link imu
- added link imu_link; visual box size=0.015 0.02 0.005
- link base_link: geometry visual box size=0.4 0.2 0.1
Joints:
- removed joint body_to_laser_frame
- removed joint laser_frame_to_imu
- added joint imu_joint: type fixed, parent base_link, child imu_link, origin xyz=0.18 0.05 -0.075 rpy=0 0 0
- added joint lidar_joint: type fixed, parent base_link, child laser, origin xyz=0.18 0 -0.075 rpy=3.14159 0 3.14159
- joint base_footprint_joint: origin xyz=0 0 0.5 rpy=0 0 0 -> xyz=0 0 0.3 rpy=0 0 0

Commit message: used internal inverted command in lidar package and reflected that inthe robot urdf

File: autonomous_litter_bot_package/urdf/robot.urdf (robot description, URDF)
Before this commit: robot go1_robot, 4 links, 3 joints
Joints:
- joint lidar_joint: origin xyz=0.18 0 -0.075 rpy=3.14159 0 3.14159 -> xyz=0.18 0 -0.075 rpy=0 0 3.14159

Commit message: Add new launch files, update URDF and setup, add unitree legged messages package

File: autonomous_litter_bot_package/urdf/robot.urdf (robot description, URDF)
Before this commit: robot go1_robot, 4 links, 3 joints
Links:
- link base_link: geometry visual box size=0.5334 0.2032 0.127
Joints:
- joint base_footprint_joint: origin xyz=0 0 0.3 rpy=0 0 0 -> xyz=0 0 0.3175 rpy=0 0 0
- joint lidar_joint: origin xyz=0.18 0 -0.075 rpy=0 0 3.14159 -> xyz=0.254 0 -0.0889 rpy=0 0 3.14159
